File: circuitos/placa-de-control/placa_de_control.kicad_sch (KiCad schematic)
At the start: 26 parts, among them J3,7IN+1 Vin+, J3,7IN-1 Vin-, J3.3a1 Screw_Terminal_01x02, J3.3b1 Screw_Terminal_01x02, J3.3c1 Screw_Terminal_01x02, J3.3out1 Screw_Terminal_01x02, J5OUT+1 Vout+, J5OUT-1 Vout-, Q1 BC337

Commit message: feat: finalizar esquematico placa de control (#80)
* refactor: borrar esquematico desactualizado

* refactor: borrar esquematico desactualizado

* feat: agregar circuito finalizado e imagenes
Parts:
- removed C1, C2: 22uF, Capacitor_THT:C_Axial_L3.8mm_D2.6mm_P7.50mm_Horizontal, symbol Device:C
- removed D1: 1N4007, Diode_THT:D_DO-41_SOD81_P10.16mm_Horizontal, symbol Diode:1N4007
- removed Q1: BC337, Package_TO_SOT_THT:TO-92_Inline, symbol Transistor_BJT:BC337
- removed Rele1: SANYOU_SRD_Form_A, Relay_THT:Relay_SPST_SANYOU_SRD_Series_Form_A, symbol Relay:SANYOU_SRD_Form_A
- added Q1: BC548, Package_TO_SOT_THT:TO-92_Inline, symbol Transistor_BJT:BC548
- added R6: 1K, Resistor_THT:R_Axial_DIN0204_L3.6mm_D1.6mm_P1.90mm_Vertical, symbol Device:R
- 3,7V_Input1, J3.3a1, J3.3b1, J3.3c1, J3.3out1, Output_Buzzer1: footprint TerminalBlock:TerminalBlock_bornier-2_P5.08mm -> TerminalBlock_Phoenix:TerminalBlock_Phoenix_MKDS-1,5-2-5.08_1x02_P5.08mm_Horizontal
- Input_MPX1: footprint TerminalBlock_Altech:Altech_AK300_1x16_P5.00mm_45-Degree -> TerminalBlock_Phoenix:TerminalBlock_Phoenix_MKDS-1,5-16_1x16_P5.00mm_Horizontal
- Input_microC1: footprint TerminalBlock:TerminalBlock_bornier-3_P5.08mm -> TerminalBlock_Phoenix:TerminalBlock_Phoenix_MKDS-1,5-3-5.08_1x03_P5.08mm_Horizontal
- LeftPinoutESP32: value Conn_01x18_Female_Right -> Conn_01x18_Female_Left; footprint Connector_PinHeader_2.54mm:PinHeader_1x18_P2.54mm_Vertical -> Connector_PinSocket_2.54mm:PinSocket_1x18_P2.54mm_Vertical
Connections:
- net 3.7V: now also 3,7V_Input1.1 (Pin_1); no longer 3,7V_Input1.2 (Pin_2)
- net 5V: now also R6.2
- net C0: now also Input_MPX1.16 (Pin_16); no longer Input_MPX1.1 (Pin_1)
- net C1: now also Input_MPX1.15 (Pin_15); no longer Input_MPX1.2 (Pin_2)
- net C10: now also Input_MPX1.6 (Pin_6); no longer Input_MPX1.11 (Pin_11)
- net C11: now also Input_MPX1.5 (Pin_5); no longer Input_MPX1.12 (Pin_12)
- net C12: now also Input_MPX1.4 (Pin_4); no longer Input_MPX1.13 (Pin_13)
- net C13: now also Input_MPX1.3 (Pin_3); no longer Input_MPX1.14 (Pin_14)
- net C14: now also Input_MPX1.2 (Pin_2); no longer Input_MPX1.15 (Pin_15)
- net C15: now also Input_MPX1.1 (Pin_1); no longer Input_MPX1.16 (Pin_16)
- net C2: now also Input_MPX1.14 (Pin_14); no longer Input_MPX1.3 (Pin_3)
- net C3: now also Input_MPX1.13 (Pin_13); no longer Input_MPX1.4 (Pin_4)
- net C4: now also Input_MPX1.12 (Pin_12); no longer Input_MPX1.5 (Pin_5)
- net C5: now also Input_MPX1.11 (Pin_11); no longer Input_MPX1.6 (Pin_6)
- net C6: now also Input_MPX1.10 (Pin_10); no longer Input_MPX1.7 (Pin_7)
- net C7: now also Input_MPX1.9 (Pin_9); no longer Input_MPX1.8 (Pin_8)
- net C8: now also Input_MPX1.8 (Pin_8); no longer Input_MPX1.9 (Pin_9)
- net C9: now also Input_MPX1.7 (Pin_7); no longer Input_MPX1.10 (Pin_10)
- net GND: now also 3,7V_Input1.2 (Pin_2), J3.3a1.2 (Pin_2), J3.3b1.2 (Pin_2), J3.3c1.2 (Pin_2), Q1.3 (E); no longer 3,7V_Input1.1 (Pin_1), J3.3a1.1 (Pin_1), J3.3b1.1 (Pin_1), J3.3c1.1 (Pin_1), Output_Buzzer1.1 (Pin_1)
- net GPIO13: now also R4.1; no longer R4.2
- net GPIO15: now also R5.1, RightPinoutMPX1.8 (Pin_8); no longer RightPinoutMPX1.7 (Pin_7)
- net GPIO16: now also RightPinoutMPX1.5 (Pin_5); no longer RightPinoutMPX1.4 (Pin_4)
- net GPIO18: now also R3.1; no longer R1.1
- net GPIO2: now also RightPinoutMPX1.7 (Pin_7); no longer RightPinoutMPX1.6 (Pin_6)
- net GPIO21: now also R1.1; no longer R3.1
- net GPIO25: now also J3.3a1.1 (Pin_1); no longer J3.3a1.2 (Pin_2)
- net GPIO26: now also J3.3b1.1 (Pin_1); no longer J3.3b1.2 (Pin_2)
- net GPIO27: now also J3.3c1.1 (Pin_1); no longer J3.3c1.2 (Pin_2)
- net GPIO4: now also RightPinoutMPX1.6 (Pin_6); no longer RightPinoutMPX1.5 (Pin_5)
- net at Output_Buzzer1.2 (Pin_2): now also R6.1
- net GPIO17: now reaches RightPinoutESP32.9 (Pin_9)
- net GPIO17: now also RightPinoutMPX1.4 (Pin_4)
- removed net GPIO0: R5.1, RightPinoutESP32.14 (Pin_14), RightPinoutMPX1.8 (Pin_8)
- new net: Output_Buzzer1.1 (Pin_1), Q1.1 (C)
- new net: Q1.2 (B), R4.2
Other:
- note added: "Módulo Rele"
- moved on the sheet: 3,7V_Input1, Input_MPX1, J3.3a1, J3.3b1, J3.3c1, R1, R2, R3
